File: board/radius.sch (KiCad schematic (older format))
At the start: 11 parts, among them IC1 STM8S003F3P, P1 CONN_01X04, P2 CONN_01X10, U1 CH340G, U2 LM2931AZ-3.3/5.0, Y1 Crystal

Commit message: Updates capacitor values.
Parts:
- C1: value 0.1 µF -> 10 µF
Changed lines of the file:
@@
 P 8700 5150
 F 0 "C1" H 8725 5250 50  0000 L CNN
-F 1 "0.1 µF" H 8725 5050 50  0000 L CNN
+F 1 "10 µF" H 8725 5050 50  0000 L CNN
 F 2 "Capacitors_SMD:C_0603_HandSoldering" H 8738 5000 30  0001 C CNN
 F 3 "" H 8700 5150 60  0000 C CNN
